File: kicad/exercise 4-1/exercise 4.kicad_sch (KiCad schematic)
At the start: 6 parts

Commit message: done
Parts:
- C1: footprint (none) -> Capacitor_THT:C_Radial_D5.0mm_H5.0mm_P2.00mm
- D1: footprint (none) -> LED_THT:LED_D5.0mm
- R1, R2: footprint (none) -> Resistor_THT:R_Axial_DIN0516_L15.5mm_D5.0mm_P20.32mm_Horizontal
- SW1: renamed from SW?; footprint (none) -> Button_Switch_THT:SW_E-Switch_EG1224_SPDT_Angled
- V1: renamed from V; footprint (none) -> Connector_JST:JST_PH_B2B-PH-K_1x02_P2.00mm_Vertical
Other:
- moved on the sheet: D1, R1, V1
Changed lines of the file:
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@@
 (kicad_sch (version 20211123) (generator eeschema)
   (paper "A4")
+  (junction (at 177.8 116.84) (diameter 0) (color 0 0 0 0)
+  )
+  (junction (at 177.8 100.33) (diameter 0) (color 0 0 0 0)
+  )
   (junction (at 177.8 83.82) (diameter 0) (color 0 0 0 0)
   )
-  (junction (at 177.8 113.03) (diameter 0) (color 0 0 0 0)
+  (junction (at 193.04 113.03) (diameter 0) (color 0 0 0 0)
   )
-  (wire (pts (xy 177.8 100.33) (xy 177.8 113.03))
+  (wire (pts (xy 177.8 99.06) (xy 177.8 100.33))
     (stroke (width 0) (type default) (color 0 0 0 0))
   )
-  (wire (pts (xy 191.77 113.03) (xy 177.8 113.03))
+  (wire (pts (xy 193.04 113.03) (xy 193.04 116.84))
     (stroke (width 0) (type default) (color 0 0 0 0))
   )
-  (wire (pts (xy 154.94 81.28) (xy 151.13 81.28))
+  (wire (pts (xy 193.04 83.82) (xy 193.04 90.17))
     (stroke (width 0) (type default) (color 0 0 0 0))
   )
-  (wire (pts (xy 151.13 113.03) (xy 177.8 113.03))
+  (wire (pts (xy 149.86 99.06) (xy 149.86 116.84))
+    (stroke (width 0) (type default) (color 0 0 0 0))
+  )
+  (wire (pts (xy 193.04 111.76) (xy 193.04 113.03))
+    (stroke (width 0) (type default) (color 0 0 0 0))
+  )
+  (wire (pts (xy 177.8 83.82) (xy 193.04 83.82))
+    (stroke (width 0) (type default) (color 0 0 0 0))
+  )
+  (wire (pts (xy 177.8 116.84) (xy 193.04 116.84))
+    (stroke (width 0) (type default) (color 0 0 0 0))
+  )
+  (wire (pts (xy 177.8 100.33) (xy 177.8 116.84))
     (stroke (width 0) (type default) (color 0 0 0 0))
   )
@@
     (stroke (width 0) (type default) (color 0 0 0 0))
   )
+  (wire (pts (xy 149.86 81.28) (xy 154.94 81.28))
+    (stroke (width 0) (type default) (color 0 0 0 0))
+  )
+  (wire (pts (xy 149.86 81.28) (xy 149.86 96.52))
+    (stroke (width 0) (type default) (color 0 0 0 0))
+  )
   (wire (pts (xy 175.26 83.82) (xy 177.8 83.82))
     (stroke (width 0) (type default) (color 0 0 0 0))
   )
-  (wire (pts (xy 151.13 99.06) (xy 151.13 113.03))
-    (stroke (width 0) (type default) (color 0 0 0 0))
-  )
-  (wire (pts (xy 177.8 83.82) (xy 191.77 83.82))
-    (stroke (width 0) (type default) (color 0 0 0 0))
-  )
-  (wire (pts (xy 151.13 81.28) (xy 151.13 96.52))
-    (stroke (width 0) (type default) (color 0 0 0 0))
-  )
-  (wire (pts (xy 191.77 83.82) (xy 191.77 92.71))
+  (wire (pts (xy 149.86 116.84) (xy 177.8 116.84))
     (stroke (width 0) (type default) (color 0 0 0 0))
   )
@@
     (stroke (width 0) (type default) (color 0 0 0 0))
   )
-  (wire (pts (xy 191.77 100.33) (xy 191.77 105.41))
+  (wire (pts (xy 193.04 97.79) (xy 193.04 105.41))
     (stroke (width 0) (type default) (color 0 0 0 0))
   )
@@
       (effects (font (size 1.27 1.27)) (justify left))
     )
-    (property "Footprint" "" (id 2) (at 178.7652 100.33 0)
+    (property "Footprint" "Capacitor_THT:C_Radial_D5.0mm_H5.0mm_P2.00mm" (id 2) (at 178.7652 100.33 0)
       (effects (font (size 1.27 1.27)) hide)
     )
@@
     (pin "2")
   )
-  (symbol (lib_id "Device:LED") (at 191.77 109.22 90) (unit 1)
+  (symbol (lib_id "Device:LED") (at 193.04 109.22 90) (unit 1)
     (in_bom yes) (on_board yes) (fields_autoplaced)
-    (property "Reference" "D1" (id 0) (at 195.58 109.5374 90)
+    (property "Reference" "D1" (id 0) (at 196.85 109.5374 90)
       (effects (font (size 1.27 1.27)) (justify right))
     )
-    (property "Value" "LED" (id 1) (at 195.58 112.0774 90)
+    (property "Value" "LED" (id 1) (at 196.85 112.0774 90)
       (effects (font (size 1.27 1.27)) (justify right))
     )
-    (property "Footprint" "" (id 2) (at 191.77 109.22 0)
+    (property "Footprint" "LED_THT:LED_D5.0mm" (id 2) (at 193.04 109.22 0)
       (effects (font (size 1.27 1.27)) hide)
     )
-    (property "Datasheet" "~" (id 3) (at 191.77 109.22 0)
+    (property "Datasheet" "~" (id 3) (at 193.04 109.22 0)
       (effects (font (size 1.27 1.27)) hide)
     )
@@
     (property "Reference" "R2" (id 0) (at 158.75 74.93 90))
     (property "Value" "2.2K" (id 1) (at 158.75 77.47 90))
-    (property "Footprint" "" (id 2) (at 158.75 83.058 90)
+    (property "Footprint" "Resistor_THT:R_Axial_DIN0516_L15.5mm_D5.0mm_P20.32mm_Horizontal" (id 2) (at 158.75 83.058 90)
       (effects (font (size 1.27 1.27)) hide)
     )
@@
     (pin "2")
   )
-  (symbol (lib_id "Connector:Conn_01x02_Male") (at 146.05 96.52 0) (unit 1)
+  (symbol (lib_id "Connector:Conn_01x02_Male") (at 144.78 96.52 0) (unit 1)
     (in_bom yes) (on_board yes) (fields_autoplaced)
-    (property "Reference" "V" (id 0) (at 146.685 91.44 0))
-    (property "Value" "9 V" (id 1) (at 146.685 93.98 0))
-    (property "Footprint" "" (id 2) (at 146.05 96.52 0)
+    (property "Reference" "V1" (id 0) (at 145.415 91.44 0))
+    (property "Value" "9 V" (id 1) (at 145.415 93.98 0))
+    (property "Footprint" "Connector_JST:JST_PH_B2B-PH-K_1x02_P2.00mm_Vertical" (id 2) (at 144.78 96.52 0)
       (effects (font (size 1.27 1.27)) hide)
     )
-    (property "Datasheet" "~" (id 3) (at 146.05 96.52 0)
+    (property "Datasheet" "~" (id 3) (at 144.78 96.52 0)
       (effects (font (size 1.27 1.27)) hide)
     )
@@
   (symbol (lib_id "Switch:SW_SPDT") (at 170.18 81.28 0) (unit 1)
     (in_bom yes) (on_board yes) (fields_autoplaced)
-    (property "Reference" "SW?" (id 0) (at 170.18 73.66 0))
+    (property "Reference" "SW1" (id 0) (at 170.18 73.66 0))
     (property "Value" "SW_SPDT" (id 1) (at 170.18 76.2 0))
-    (property "Footprint" "" (id 2) (at 170.18 81.28 0)
+    (property "Footprint" "Button_Switch_THT:SW_E-Switch_EG1224_SPDT_Angled" (id 2) (at 170.18 81.28 0)
       (effects (font (size 1.27 1.27)) hide)
     )
@@
     (pin "3")
   )
-  (symbol (lib_id "Device:R") (at 191.77 96.52 0) (unit 1)
+  (symbol (lib_id "Device:R") (at 193.04 93.98 0) (unit 1)
     (in_bom yes) (on_board yes) (fields_autoplaced)
-    (property "Reference" "R1" (id 0) (at 194.31 95.2499 0)
+    (property "Reference" "R1" (id 0) (at 195.58 92.7099 0)
       (effects (font (size 1.27 1.27)) (justify left))
     )
-    (property "Value" "20K" (id 1) (at 194.31 97.7899 0)
+    (property "Value" "20K" (id 1) (at 195.58 95.2499 0)
       (effects (font (size 1.27 1.27)) (justify left))
     )
-    (property "Footprint" "" (id 2) (at 189.992 96.52 90)
+    (property "Footprint" "Resistor_THT:R_Axial_DIN0516_L15.5mm_D5.0mm_P20.32mm_Horizontal" (id 2) (at 191.262 93.98 90)
       (effects (font (size 1.27 1.27)) hide)
     )
-    (property "Datasheet" "~" (id 3) (at 191.77 96.52 0)
+    (property "Datasheet" "~" (id 3) (at 193.04 93.98 0)
       (effects (font (size 1.27 1.27)) hide)
     )
@@
   (symbol_instances
     (path "/39544411-91b8-4cf7-ad8b-a1816153ba51"
-      (reference "C1") (unit 1) (value "4.7 uF") (footprint "")
+      (reference "C1") (unit 1) (value "4.7 uF") (footprint "Capacitor_THT:C_Radial_D5.0mm_H5.0mm_P2.00mm")
     )
     (path "/433b0fa4-341b-4be3-af5a-da158b3eb893"
-      (reference "D1") (unit 1) (value "LED") (footprint "")
+      (reference "D1") (unit 1) (value "LED") (footprint "LED_THT:LED_D5.0mm")
     )
     (path "/fd7757b9-f36d-4551-a9a3-a6b646006538"
-      (reference "R1") (unit 1) (value "20K") (footprint "")
+      (reference "R1") (unit 1) (value "20K") (footprint "Resistor_THT:R_Axial_DIN0516_L15.5mm_D5.0mm_P20.32mm_Horizontal")
     )
     (path "/5e1cffdf-0adf-4e33-93f4-882e06420b22"
-      (reference "R2") (unit 1) (value "2.2K") (footprint "")
+      (reference "R2") (unit 1) (value "2.2K") (footprint "Resistor_THT:R_Axial_DIN0516_L15.5mm_D5.0mm_P20.32mm_Horizontal")
     )
     (path "/d4ec28b1-7a1f-493f-9417-64c9337fdf67"
-      (reference "SW?") (unit 1) (value "SW_SPDT") (footprint "")
+      (reference "SW1") (unit 1) (value "SW_SPDT") (footprint "Button_Switch_THT:SW_E-Switch_EG1224_SPDT_Angled")
     )
     (path "/969aabff-58da-457d-91be-8cc20d40150e"
-      (reference "V") (unit 1) (value "9 V") (footprint "")
+      (reference "V1") (unit 1) (value "9 V") (footprint "Connector_JST:JST_PH_B2B-PH-K_1x02_P2.00mm_Vertical")
     )
   )
